File: Controller v2.brd (EAGLE design)
At the start: 100 x 80 mm, 76 parts, among them IC1 MCP23017ML, Q1 AOD4184A, Q2 AOD4184A, Q3 AOD4184A, Q4 AOD4184A, U1 ADS1115IDGST, U2 ADS1115IDGST, U3 ULN2803ADWRG4, X1 53048-03, X10 53048-04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

Commit message: Updated board
Parts:
- removed JP1: (no value), adafruit:2X04
- removed JP3, JP4, JP5: (no value), pinhead:1X02
- added C12, C13: 47uF, rcl:C0805K
- added R13: 4.32K, rcl:R0402
- added R14: 10K, rcl:R0402
- added U4: TPSM53604RDAR, TPSM53604:B3QFN14_RDA_TEX
- C1, C2, C3, C7, C8: device microbuilder:0805-NO -> rcl:C0603
- C10, C11, C6, C9: device microbuilder:0805-NO -> rcl:C0805K
- C4, C5: value 100uF -> 10uF; device microbuilder:0805-NO -> rcl:C0805K
- D8: device microbuilder:CHIPLED_0805_NOOUTLINE -> adafruit:CHIPLED_0805
- JP2: value (none) -> 3.3V; device pinhead:1X02 -> jumper:JP4Q
- R1, R12, R2: device microbuilder:0603-NO -> rcl:R0805
- R11: device microbuilder:0603-NO -> rcl:R0603
- moved JP2 24.7 mm to (42.5, 52.1), turned to 180 degrees
- moved C5 3.42 mm to (19.7, 71.1), turned to 0 degrees
- moved C4 0.90 mm to (19.7, 69.2), turned to 0 degrees
Connections:
- new net N$29: R13.2, R14.2, U4.9
- net +12V: now also U4.1, U4.14, U4.2; no longer JP2.1, JP2.2
- net 3.3V: now also C12.1, C13.1, JP2.7, JP2.8, R14.1, U4.7, U4.8; no longer JP1.1, JP1.2, JP4.1, JP4.2
- net GND: now also C12.2, C13.2, JP2.1, JP2.2, R13.1, U4.12, U4.15; no longer JP1.7, JP1.8, JP3.1, JP3.2, JP5.1, JP5.2
- net SCL: now also JP2.5, JP2.6; no longer JP1.3, JP1.4
- net SDA: now also JP2.3, JP2.4; no longer JP1.5, JP1.6
Routing:
- net 3.3V: track 426.1 -> 464.9 mm, vias 6 -> 1
- net +12V: track 132.8 -> 143.8 mm
- net N$29: track 0.00 -> 3.16 mm
- net GND: track 189.2 -> 191.4 mm, vias 132 -> 120
- net SDA: track 107.4 -> 108.5 mm
- removed copper zone on layer 1, net 3.3V
- removed copper zone on layer 16, net 3.3V
