File: Controller v2.sch (EAGLE design)
At the start: 76 parts, among them IC1 MCP23017ML, Q1 AOD4184A, Q2 AOD4184A, Q3 AOD4184A, Q4 AOD4184A, U1 ADS1115IDGST, U2 ADS1115IDGST, U3 ULN2803ADWRG4, X1 53048-03, X10 53048-04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

Commit message: Updated board
Parts:
- removed JP1: (no value), adafruit:PINHD-2X4
- removed JP3, JP4, JP5: (no value), pinhead:PINHD-1X2
- added C12, C13: 47uF, rcl:C-EUC0805K
- added R13: 4.32K, rcl:R-EU_R0402
- added R14: 10K, rcl:R-EU_R0402
- added U4: TPSM53604RDAR, TPSM53604:TPSM53604RDAR
- C1, C2, C3, C7, C8: device microbuilder:CAP_CERAMIC0805-NOOUTLINE -> rcl:C-EUC0603
- C10, C11, C6, C9: device microbuilder:CAP_CERAMIC0805-NOOUTLINE -> rcl:C-EUC0805K
- C4, C5: value 100uF -> 10uF; device microbuilder:CAP_CERAMIC0805-NOOUTLINE -> rcl:C-EUC0805K
- D8: device microbuilder:LED0805_NOOUTLINE -> adafruit:LEDCHIPLED_0805
- JP2: value (none) -> 3.3V; device pinhead:PINHD-1X2 -> jumper:JP4QE
- R1, R12, R2: device microbuilder:RESISTOR_0603_NOOUT -> rcl:R-EU_R0805
- R11: device microbuilder:RESISTOR_0603_NOOUT -> rcl:R-EU_R0603
Connections:
- new net N$29: R13.2, R14.2, U4.FB
- net +12V: now also U4.EN, U4.VIN, U4.VIN_2; no longer JP2.1, JP2.2
- net 3.3V: now also C12.1, C13.1, JP2-4.1, JP2-4.2, R14.1, U4.VOUT, U4.VOUT_2; no longer JP1.1, JP1.2, JP4.1, JP4.2
- net GND: now also C12.2, C13.2, JP2-1.1, JP2-1.2, R13.1, U4.AGND, U4.PGND; no longer JP1.7, JP1.8, JP3.1, JP3.2, JP5.1, JP5.2
- net SCL: now also JP2-3.1, JP2-3.2; no longer JP1.3, JP1.4
- net SDA: now also JP2-2.1, JP2-2.2; no longer JP1.5, JP1.6
Other:
- moved on the sheet: C1, C10, C11, C2, C3, C4, C5, C6, C7, C8, C9, D12
